Commit message: add red color

File: src/my_cobot_description/urdf/common_properties.xacro (robot description, xacro)
@@ -10,3 +10,6 @@
         <color rgba="1 1 0 1"/>
     </material>
+    <material name="red">
+        <color rgba="1 0 0 1"/>
+    </material>
 </robot>

Commit message: add macros that define inertial of box cylinder and sphere

File: src/my_cobot_description/urdf/common_properties.xacro (robot description, xacro)
@@ -13,3 +13,30 @@
         <color rgba="1 0 0 1"/>
     </material>
+    <xacro:macro name="box_inertia" params="m l w  xyz rpy">
+        <inertial>
+            <origin xyz="${xyz}" rpy="${rpy}"/>
+            <mass value="${m}" />
+            <inertia ixx="${(m/12) * (h*h + l*l)}" ixy="0" ixz="0"
+                     iyy="${(m/12) * (w*w + l*l)}" iyz="0"
+                     izz="${(m/12) * (w*w + h*h)}"/>
+        </inertial>
+    </xacro:macro>
+    <xacro:macro name="cylinder_inertia" params="m r l xyz rpy">
+        <inertial>
+            <origin xyz="${xyz}" rpy="${rpy}"/>
+            <mass value="${m}"/>
+            <inertia ixx="${(m/12)*(3*r*r + l*l)}" ixy="0" ixz="0"
+                     iyy="${(m/12)*(3*r*r + l*l)}" iyz="0"
+                     izz="${m*r*r/2.0}"/>
+        </inertial>
+    </xacro:macro>
+    <xacro:macro name="sphere_inertia" params="m r xyz rpy">
+        <inertial>
+            <origin xyz="${xyz}" rpy="${rpy}"/>
+            <mass value="${m}"/>
+            <inertia ixx="${(2/5)*m*r*r}" ixy="0" ixz="0"
+                     iyy="${(2/5)*m*r*r}" iyz="0"
+                     izz="${(2/5)*m*r*r}"/>
+        </inertial>
+    </xacro:macro>
 </robot>
