Commit message: add the gripper link

File: src/my_cobot_description/urdf/cobot_arm.xacro (robot description, xacro)
@@ -62,4 +62,13 @@
         </visual>
     </link>
+    <link name="gripper">
+        <visual>
+            <geometry>
+                <sphere radius="${solid_radius * 0.8}"/>
+            </geometry>
+            <origin xyz="0 0 0" rpy="0 0 0"/>
+            <material name="red"/>
+        </visual>
+    </link>
     <joint name="base_joint" type="fixed">
         <parent link="base_footprint"/>
@@ -95,3 +104,8 @@
         <axis xyz="0 1 0"/>
     </joint>
+    <joint name="end_effector" type="fixed">
+        <parent link="link_3"/>
+        <child link="gripper"/>
+        <origin xyz="0 0 ${joint_length_2}" rpy="0 0 0"/>
+    </joint>
 </robot>

Commit message: add collusion to each link

File: src/my_cobot_description/urdf/cobot_arm.xacro (robot description, xacro)
@@ -15,4 +15,10 @@
             <material name="grey"/>
         </visual>
+        <collision>
+            <geometry>
+                <box size="${base_size} ${base_size} ${base_height}"/>
+            </geometry>
+            <origin xyz="0 0 ${base_height/2}" rpy="0 0 0"/>
+        </collision>
     </link>
     <link name="base_footprint"/>
@@ -25,4 +31,10 @@
             <material name="blue"/>
         </visual>
+        <collision>
+            <geometry>
+                <cylinder radius="${joint_radius_1}" length="${joint_length_1}"/>
+            </geometry>
+            <origin xyz="0 0 ${joint_length_1/2}" rpy="0 0 0 "/>
+        </collision>
     </link>
     <link name="solid_1">
@@ -34,4 +46,10 @@
             <material name="yellow"/>
         </visual>
+        <collision>
+            <geometry>
+                <sphere radius="${solid_radius}"/>
+            </geometry>
+            <origin xyz="0 0 0" rpy="0 0 0"/>
+        </collision>
     </link>
     <link name="link_2">
@@ -43,4 +61,10 @@
             <material name="blue"/>
         </visual>
+        <collision>
+            <geometry>
+                <cylinder radius="${joint_radius_1 * 0.8}" length="${joint_length_2}"/>
+            </geometry>
+            <origin xyz="0 0 ${joint_length_2/2}" rpy="0 0 0"/>
+        </collision>
     </link>
     <link name="solid_2">
@@ -52,4 +76,10 @@
             <material name="yellow"/>
         </visual>
+        <collision>
+            <geometry>
+                <sphere radius="${solid_radius}"/>
+            </geometry>
+            <origin xyz="0 0 0" rpy="0 0 0"/>
+        </collision>
     </link>
     <link name="link_3">
@@ -61,4 +91,10 @@
             <material name="blue"/>
         </visual>
+        <collision>
+            <geometry>
+                <cylinder radius="${joint_radius_1 * 0.6}" length="${joint_length_2}"/>
+            </geometry>
+            <origin xyz="0 0 ${joint_length_2/2}" rpy="0 0 0"/>
+        </collision>
     </link>
     <link name="gripper">
@@ -70,4 +106,10 @@
             <material name="red"/>
         </visual>
+        <collision>
+            <geometry>
+                <sphere radius="${solid_radius * 0.8}"/>
+            </geometry>
+            <origin xyz="0 0 0" rpy="0 0 0"/>
+        </collision>
     </link>
     <joint name="base_joint" type="fixed">

Commit message: add inertia for each link

File: src/my_cobot_description/urdf/cobot_arm.xacro (robot description, xacro)
@@ -21,4 +21,6 @@
             <origin xyz="0 0 ${base_height/2}" rpy="0 0 0"/>
         </collision>
+        <xacro:box_inertia m="5.0" l="${2*base_size}" w="${2*base_size}" h="${2*base_height}"
+                           xyz="0 0 ${base_height/2}" rpy="0 0 0"/>
     </link>
     <link name="base_footprint"/>
@@ -35,6 +37,8 @@
                 <cylinder radius="${joint_radius_1}" length="${joint_length_1}"/>
             </geometry>
-            <origin xyz="0 0 ${joint_length_1/2}" rpy="0 0 0 "/>
+            <origin xyz="0 0 ${joint_length_1/2}" rpy="0 0 0"/>
         </collision>
+        <xacro:cylinder_inertia m="1.0" r="${2*joint_radius_1}" l="${2*joint_length_1}"
+                                xyz="0 0 ${joint_length_1/2}" rpy="0 0 0"/>
     </link>
     <link name="solid_1">
@@ -52,4 +56,5 @@
             <origin xyz="0 0 0" rpy="0 0 0"/>
         </collision>
+        <xacro:sphere_inertia m="0.5" r="${2*solid_radius}" xyz="0 0 0" rpy="0 0 0"/>
     </link>
     <link name="link_2">
@@ -67,4 +72,6 @@
             <origin xyz="0 0 ${joint_length_2/2}" rpy="0 0 0"/>
         </collision>
+        <xacro:cylinder_inertia m="1.0" r="${2*joint_radius_1 * 0.8}" l="${2*joint_length_2}"
+                                xyz="0 0 ${joint_length_2/2}" rpy="0 0 0"/>
     </link>
     <link name="solid_2">
@@ -82,4 +89,5 @@
             <origin xyz="0 0 0" rpy="0 0 0"/>
         </collision>
+        <xacro:sphere_inertia m="0.5" r="${2*solid_radius}" xyz="0 0 0" rpy="0 0 0"/>
     </link>
     <link name="link_3">
@@ -97,4 +105,6 @@
             <origin xyz="0 0 ${joint_length_2/2}" rpy="0 0 0"/>
         </collision>
+        <xacro:cylinder_inertia m="1.0" r="${2*joint_radius_1 * 0.6}" l="${2*joint_length_2}"
+                                xyz="0 0 ${joint_length_2/2}" rpy="0 0 0"/>
     </link>
     <link name="gripper">
@@ -112,4 +122,5 @@
             <origin xyz="0 0 0" rpy="0 0 0"/>
         </collision>
+        <xacro:sphere_inertia m="0.5" r="${2*solid_radius * 0.8}" xyz="0 0 0" rpy="0 0 0"/>
     </link>
     <joint name="base_joint" type="fixed">

File: src/my_cobot_description/urdf/common_properties.xacro (robot description, xacro)
@@ -13,5 +13,5 @@
         <color rgba="1 0 0 1"/>
     </material>
-    <xacro:macro name="box_inertia" params="m l w  xyz rpy">
+    <xacro:macro name="box_inertia" params="m l w h xyz rpy">
         <inertial>
             <origin xyz="${xyz}" rpy="${rpy}"/>
