Commit message: add gazebo color for the robot and change joint type to revolute

File: src/my_cobot_description/urdf/cobot.urdf.xacro (robot description, xacro)
@@ -3,3 +3,4 @@
     <xacro:include filename="common_properties.xacro"/>
     <xacro:include filename="cobot_arm.xacro"/>
+    <xacro:include filename="cobot_arm_gazebo.xacro"/>
 </robot>

File: src/my_cobot_description/urdf/cobot_arm.xacro (robot description, xacro)
@@ -21,5 +21,5 @@
             <origin xyz="0 0 ${base_height/2}" rpy="0 0 0"/>
         </collision>
-        <xacro:box_inertia m="5.0" l="${2*base_size}" w="${2*base_size}" h="${2*base_height}"
+        <xacro:box_inertia m="50" l="${2*base_size}" w="${2*base_size}" h="${2*base_height}"
                            xyz="0 0 ${base_height/2}" rpy="0 0 0"/>
     </link>
@@ -129,9 +129,11 @@
         <origin xyz="0 0 0" rpy="0 0 0"/>
     </joint>
-    <joint name="base_joint_1" type="continuous">
+    <joint name="base_joint_1" type="revolute">
         <parent link="base_link"/>
         <child link="link_1"/>
         <origin xyz="0 0 ${base_height}" rpy="0 0 0"/>
         <axis xyz="0 0 1"/>
+        <limit lower="0" upper="${pi/2}" effort="100" velocity="100"/>
+        <dynamics friction="0.05" damping="0.1"/>
     </joint>
     <joint name="joint_1_solid" type="fixed">
@@ -140,9 +142,11 @@
         <origin xyz="0 0 ${joint_length_1}" rpy="0 0 0"/>
     </joint>
-    <joint name="solid_1_joint" type="continuous">
+    <joint name="solid_1_joint" type="revolute">
         <parent link="solid_1"/>
         <child link="link_2"/>
         <origin xyz="0 0 0" rpy="0 0 0"/>
         <axis xyz="0 1 0"/>
+        <limit lower="0" upper="${pi/2}" effort="100" velocity="100"/>
+        <dynamics friction="0.05" damping="0.1"/>
     </joint>
     <joint name="joint_2_solid" type="fixed">
@@ -151,9 +155,11 @@
         <origin xyz="0 0 ${joint_length_2}" rpy="0 0 0"/>
     </joint>
-    <joint name="solid_2_joint" type="continuous">
+    <joint name="solid_2_joint" type="revolute">
         <parent link="solid_2"/>
         <child link="link_3"/>
         <origin xyz="0 0 0" rpy="0 0 0"/>
         <axis xyz="0 1 0"/>
+        <limit lower="0" upper="${pi/2}" effort="100" velocity="100"/>
+        <dynamics friction="0.05" damping="0.1"/>
     </joint>
     <joint name="end_effector" type="fixed">
