Commit message: increate the friciton and damping of the joints

File: install/my_cobot_description/share/my_cobot_description/urdf/cobot_arm.xacro (robot description, xacro)
@@ -135,5 +135,5 @@
         <axis xyz="0 0 1"/>
         <limit lower="0" upper="${pi/2}" effort="100" velocity="100"/>
-        <dynamics friction="0.05" damping="0.1"/>
+        <dynamics friction="010" damping="10"/>
     </joint>
     <joint name="joint_1_solid" type="fixed">
@@ -148,5 +148,5 @@
         <axis xyz="0 1 0"/>
         <limit lower="0" upper="${pi/2}" effort="100" velocity="100"/>
-        <dynamics friction="0.05" damping="0.1"/>
+        <dynamics friction="100" damping="100"/>
     </joint>
     <joint name="joint_2_solid" type="fixed">
@@ -161,5 +161,5 @@
         <axis xyz="0 1 0"/>
         <limit lower="0" upper="${pi/2}" effort="100" velocity="100"/>
-        <dynamics friction="0.05" damping="0.1"/>
+        <dynamics friction="100" damping="100"/>
     </joint>
     <joint name="end_effector" type="fixed">

File: install/my_cobot_description/share/my_cobot_description/urdf/cobot_arm_gazebo.xacro (robot description, xacro)
@@ -22,3 +22,16 @@
         <material>Gazebo/Red</material>
     </gazebo>
+    <gazebo>
+        <plugin name="gazebo_ros_joint_state_publisher"
+        filename="libgazebo_ros_joint_state_publisher.so">
+            <update_rate>10</update_rate>
+            <joint_name>base_joint_1</joint_name>
+            <joint_name>solid_1_joint</joint_name>
+            <joint_name>solid_2_joint</joint_name>
+        </plugin>
+        <plugin name="gazebo_ros_joint_pose_trajectory"
+            filename="libgazebo_ros_joint_pose_trajectory.so">
+            <update_rate>20</update_rate>
+        </plugin>
+    </gazebo>
 </robot>

Commit message: add inverse kinematic function

File: install/my_cobot_description/share/my_cobot_description/urdf/cobot_arm.xacro (robot description, xacro)
@@ -134,6 +134,6 @@
         <origin xyz="0 0 ${base_height}" rpy="0 0 0"/>
         <axis xyz="0 0 1"/>
-        <limit lower="0" upper="${pi/2}" effort="100" velocity="100"/>
-        <dynamics friction="010" damping="10"/>
+        <limit lower="${-pi/2}" upper="${pi/2}" effort="100" velocity="100"/>
+        <dynamics friction="1000" damping="1000"/>
     </joint>
     <joint name="joint_1_solid" type="fixed">
@@ -147,6 +147,6 @@
         <origin xyz="0 0 0" rpy="0 0 0"/>
         <axis xyz="0 1 0"/>
-        <limit lower="0" upper="${pi/2}" effort="100" velocity="100"/>
-        <dynamics friction="100" damping="100"/>
+        <limit lower="${-pi/2}" upper="${pi/2}" effort="100" velocity="100"/>
+        <dynamics friction="1000" damping="1000"/>
     </joint>
     <joint name="joint_2_solid" type="fixed">
@@ -160,6 +160,6 @@
         <origin xyz="0 0 0" rpy="0 0 0"/>
         <axis xyz="0 1 0"/>
-        <limit lower="0" upper="${pi/2}" effort="100" velocity="100"/>
-        <dynamics friction="100" damping="100"/>
+        <limit lower="${-pi/2}" upper="${5*pi/6}" effort="100" velocity="100"/>
+        <dynamics friction="1000" damping="1000"/>
     </joint>
     <joint name="end_effector" type="fixed">

Commit message: add inverse kinematics for the third link

File: install/my_cobot_description/share/my_cobot_description/urdf/cobot_arm.xacro (robot description, xacro)
@@ -134,5 +134,5 @@
         <origin xyz="0 0 ${base_height}" rpy="0 0 0"/>
         <axis xyz="0 0 1"/>
-        <limit lower="${-pi/2}" upper="${pi/2}" effort="100" velocity="100"/>
+        <limit lower="${-pi}" upper="${pi}" effort="100" velocity="100"/>
         <dynamics friction="1000" damping="1000"/>
     </joint>
@@ -147,5 +147,5 @@
         <origin xyz="0 0 0" rpy="0 0 0"/>
         <axis xyz="0 1 0"/>
-        <limit lower="${-pi/2}" upper="${pi/2}" effort="100" velocity="100"/>
+        <limit lower="${-pi}" upper="${pi}" effort="100" velocity="100"/>
         <dynamics friction="1000" damping="1000"/>
     </joint>
@@ -160,5 +160,5 @@
         <origin xyz="0 0 0" rpy="0 0 0"/>
         <axis xyz="0 1 0"/>
-        <limit lower="${-pi/2}" upper="${5*pi/6}" effort="100" velocity="100"/>
+        <limit lower="${-pi}" upper="${pi}" effort="100" velocity="100"/>
         <dynamics friction="1000" damping="1000"/>
     </joint>

Commit message: fixed joint orientation to elbow down

File: install/my_cobot_description/share/my_cobot_description/urdf/cobot_arm.xacro (robot description, xacro)
@@ -4,5 +4,5 @@
     <xacro:property name="base_size" value="0.4" />
     <xacro:property name="joint_radius_1" value="0.1" />
-    <xacro:property name="joint_length_1" value="0.3" />
+    <xacro:property name="joint_length_1" value="0.8" />
     <xacro:property name="joint_length_2" value="0.8"/>
     <xacro:property name="solid_radius" value="0.15"/>
@@ -145,5 +145,5 @@
         <parent link="solid_1"/>
         <child link="link_2"/>
-        <origin xyz="0 0 0" rpy="0 0 0"/>
+        <origin xyz="0 0 0" rpy="0 -${pi/2} ${pi}"/>
         <axis xyz="0 1 0"/>
         <limit lower="${-pi}" upper="${pi}" effort="100" velocity="100"/>
